File: hardware/LEC032002.kicad_sch (KiCad schematic)
At the start: 64 parts, among them J1 Screw_Terminal_01x02_green, J2 Screw_Terminal_01x02_blue, J3 Screw_Terminal_01x02_blue, J4 Screw_Terminal_01x02_blue, J5 Screw_Terminal_01x02_blue, U1 ATtiny24A-SSU, U2 78L05G-AB3-R, U3 MP6515, U4 LTV-814S-TA1, U5 LTV-814S-TA1

Commit message: Fix part placement
Parts:
- RV1, RV2, RV3, RV4: JLCPCB_CORRECTION 1.27;0;0 -> 0;-1.27;0
- U1, U3, U4, U5: JLCPCB_CORRECTION 0;0;90 -> 0;0;270
Changed lines of the file:
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@@
       (effects (font (size 1.27 1.27)) hide)
     )
-    (property "JLCPCB_CORRECTION" "0;0;90" (id 6) (at 54.61 90.17 0)
+    (property "JLCPCB_CORRECTION" "0;0;270" (id 6) (at 54.61 90.17 0)
       (effects (font (size 1.27 1.27)) hide)
     )
@@
       (effects (font (size 1.27 1.27)) hide)
     )
-    (property "JLCPCB_CORRECTION" "1.27;0;0" (id 7) (at 153.67 105.41 0)
+    (property "JLCPCB_CORRECTION" "0;-1.27;0" (id 7) (at 153.67 105.41 0)
       (effects (font (size 1.27 1.27)) hide)
     )
@@
       (effects (font (size 1.27 1.27)) hide)
     )
-    (property "JLCPCB_CORRECTION" "0;0;90" (id 6) (at 106.68 163.83 0)
+    (property "JLCPCB_CORRECTION" "0;0;270" (id 6) (at 106.68 163.83 0)
       (effects (font (size 1.27 1.27)) hide)
     )
@@
       (effects (font (size 1.27 1.27)) hide)
     )
-    (property "JLCPCB_CORRECTION" "1.27;0;0" (id 7) (at 191.77 105.41 0)
+    (property "JLCPCB_CORRECTION" "0;-1.27;0" (id 7) (at 191.77 105.41 0)
       (effects (font (size 1.27 1.27)) hide)
     )
@@
       (effects (font (size 1.27 1.27)) hide)
     )
-    (property "JLCPCB_CORRECTION" "1.27;0;0" (id 7) (at 191.77 130.81 0)
+    (property "JLCPCB_CORRECTION" "0;-1.27;0" (id 7) (at 191.77 130.81 0)
       (effects (font (size 1.27 1.27)) hide)
     )
@@
       (effects (font (size 1.27 1.27)) hide)
     )
-    (property "JLCPCB_CORRECTION" "1.27;0;0" (id 7) (at 153.67 130.81 0)
+    (property "JLCPCB_CORRECTION" "0;-1.27;0" (id 7) (at 153.67 130.81 0)
       (effects (font (size 1.27 1.27)) hide)
     )
@@
       (effects (font (size 1.27 1.27)) hide)
     )
-    (property "JLCPCB_CORRECTION" "0;0;90" (id 6) (at 186.69 38.1 0)
+    (property "JLCPCB_CORRECTION" "0;0;270" (id 6) (at 186.69 38.1 0)
       (effects (font (size 1.27 1.27)) hide)
     )
@@
       (effects (font (size 1.27 1.27)) hide)
     )
-    (property "JLCPCB_CORRECTION" "0;0;90" (id 6) (at 186.69 76.2 0)
-      (effects (font (size 1.27 1.27)) hide)
-    )
+    (property "JLCPCB_CORRECTION" "0;0;270" (id 6) (at 186.69 76.2 0)
+      (effects (font (size 1.27 1.27)) hide)
+    )
